Commit message: add the package ros2_control_wujihand

File: asset_description/wuji/urdf/1.xacro (robot description, xacro)
@@ -4,6 +4,4 @@
   <xacro:arg name="mesh_pkg" default="asset_description" />
   <xacro:arg name="side" default="right" />
-  <xacro:property name="mesh_pkg" value="$(arg mesh_pkg)" />
-  <xacro:property name="side" value="$(arg side)" />
   <xacro:property name="mesh_root" value="package://${mesh_pkg}/wuji/meshes/${side}" />
   <mujoco>
@@ -51,5 +49,5 @@
   </link>
   <link
-    name="finger0_link0">
+    name="finger1_link1">
     <inertial>
       <origin
@@ -91,5 +89,5 @@
   </link>
   <joint
-    name="finger0_joint0"
+    name="finger1_joint1"
     type="revolute">
     <origin
@@ -99,5 +97,5 @@
       link="palm_link" />
     <child
-      link="finger0_link0" />
+      link="finger1_link1" />
     <axis
       xyz="-0 1 -0" />
@@ -109,5 +107,5 @@
   </joint>
   <link
-    name="finger0_link1">
+    name="finger1_link2">
     <inertial>
       <origin
@@ -149,5 +147,5 @@
   </link>
   <joint
-    name="finger0_joint1"
+    name="finger1_joint2"
     type="revolute">
     <origin
@@ -155,7 +153,7 @@
       rpy="-0.57428 -0.23677 1.8034" />
     <parent
-      link="finger0_link0" />
-    <child
-      link="finger0_link1" />
+      link="finger1_link1" />
+    <child
+      link="finger1_link2" />
     <axis
       xyz="-0 -1 -0" />
@@ -167,5 +165,5 @@
   </joint>
   <link
-    name="finger0_link2">
+    name="finger1_link3">
     <inertial>
       <origin
@@ -207,5 +205,5 @@
   </link>
   <joint
-    name="finger0_joint2"
+    name="finger1_joint3"
     type="revolute">
     <origin
@@ -213,7 +211,7 @@
       rpy="0.049049 0.017311 -1.9085" />
     <parent
-      link="finger0_link1" />
-    <child
-      link="finger0_link2" />
+      link="finger1_link2" />
+    <child
+      link="finger1_link3" />
     <axis
       xyz="0 1 0" />
@@ -225,5 +223,5 @@
   </joint>
   <link
-    name="finger0_link3">
+    name="finger1_link4">
     <inertial>
       <origin
@@ -265,5 +263,5 @@
   </link>
   <joint
-    name="finger0_joint3"
+    name="finger1_joint4"
     type="revolute">
     <origin
@@ -271,7 +269,7 @@
       rpy="0 0 0" />
     <parent
-      link="finger0_link2" />
-    <child
-      link="finger0_link3" />
+      link="finger1_link3" />
+    <child
+      link="finger1_link4" />
     <axis
       xyz="0 1 0" />
@@ -283,5 +281,5 @@
   </joint>
   <link
-    name="finger0_tip_link">
+    name="finger1_tip_link">
     <inertial>
       <origin
@@ -323,5 +321,5 @@
   </link>
   <joint
-    name="finger0_tip_fixed"
+    name="finger1_tip_fixed"
     type="fixed">
     <origin
@@ -329,12 +327,12 @@
       rpy="0 0 0" />
     <parent
-      link="finger0_link3" />
-    <child
-      link="finger0_tip_link" />
+      link="finger1_link4" />
+    <child
+      link="finger1_tip_link" />
     <axis
       xyz="0 0 0" />
   </joint>
   <link
-    name="finger1_link0">
+    name="finger2_link1">
     <inertial>
       <origin
@@ -376,5 +374,5 @@
   </link>
   <joint
-    name="finger1_joint0"
+    name="finger2_joint1"
     type="revolute">
     <origin
@@ -384,5 +382,5 @@
       link="palm_link" />
     <child
-      link="finger1_link0" />
+      link="finger2_link1" />
     <axis
       xyz="0 1 0" />
@@ -394,5 +392,5 @@
   </joint>
   <link
-    name="finger1_link1">
+    name="finger2_link2">
     <inertial>
       <origin
@@ -434,5 +432,5 @@
   </link>
   <joint
-    name="finger1_joint1"
+    name="finger2_joint2"
     type="revolute">
     <origin
@@ -440,7 +438,7 @@
       rpy="0 0 0" />
     <parent
-      link="finger1_link0" />
-    <child
-      link="finger1_link1" />
+      link="finger2_link1" />
+    <child
+      link="finger2_link2" />
     <axis
       xyz="-1 0 0" />
@@ -452,5 +450,5 @@
   </joint>
   <link
-    name="finger1_link2">
+    name="finger2_link3">
     <inertial>
       <origin
@@ -492,5 +490,5 @@
   </link>
   <joint
-    name="finger1_joint2"
+    name="finger2_joint3"
     type="revolute">
     <origin
@@ -498,7 +496,7 @@
       rpy="0 0 -0.00026861" />
     <parent
-      link="finger1_link1" />
-    <child
-      link="finger1_link2" />
+      link="finger2_link2" />
+    <child
+      link="finger2_link3" />
     <axis
       xyz="-0 1 -0" />
@@ -510,5 +508,5 @@
   </joint>
   <link
-    name="finger1_link3">
+    name="finger2_link4">
     <inertial>
       <origin
@@ -550,5 +548,5 @@
   </link>
   <joint
-    name="finger1_joint3"
+    name="finger2_joint4"
     type="revolute">
     <origin
@@ -556,7 +554,7 @@
       rpy="0 0 0" />
     <parent
-      link="finger1_link2" />
-    <child
-      link="finger1_link3" />
+      link="finger2_link3" />
+    <child
+      link="finger2_link4" />
     <axis
       xyz="-0 1 -0" />
@@ -568,5 +566,5 @@
   </joint>
   <link
-    name="finger1_tip_link">
+    name="finger2_tip_link">
     <inertial>
       <origin
@@ -608,5 +606,5 @@
   </link>
   <joint
-    name="finger1_tip_fixed"
+    name="finger2_tip_fixed"
     type="fixed">
     <origin
@@ -614,12 +612,12 @@
       rpy="0 0 0" />
     <parent
-      link="finger1_link3" />
-    <child
-      link="finger1_tip_link" />
+      link="finger2_link4" />
+    <child
+      link="finger2_tip_link" />
     <axis
       xyz="0 0 0" />
   </joint>
   <link
-    name="finger2_link0">
+    name="finger3_link1">
     <inertial>
       <origin
@@ -661,5 +659,5 @@
   </link>
   <joint
-    name="finger2_joint0"
+    name="finger3_joint1"
     type="revolute">
     <origin
@@ -669,5 +667,5 @@
       link="palm_link" />
     <child
-      link="finger2_link0" />
+      link="finger3_link1" />
     <axis
       xyz="0 1 0" />
@@ -679,5 +677,5 @@
   </joint>
   <link
-    name="finger2_link1">
+    name="finger3_link2">
     <inertial>
       <origin
@@ -719,5 +717,5 @@
   </link>
   <joint
-    name="finger2_joint1"
+    name="finger3_joint2"
     type="revolute">
     <origin
@@ -725,7 +723,7 @@
       rpy="0 0 0" />
     <parent
-      link="finger2_link0" />
-    <child
-      link="finger2_link1" />
+      link="finger3_link1" />
+    <child
+      link="finger3_link2" />
     <axis
       xyz="-1 0 0" />
@@ -737,5 +735,5 @@
   </joint>
   <link
-    name="finger2_link2">
+    name="finger3_link3">
     <inertial>
       <origin
@@ -777,5 +775,5 @@
   </link>
   <joint
-    name="finger2_joint2"
+    name="finger3_joint3"
     type="revolute">
     <origin
@@ -783,7 +781,7 @@
       rpy="0 0 -0.00026861" />
     <parent
-      link="finger2_link1" />
-    <child
-      link="finger2_link2" />
+      link="finger3_link2" />
+    <child
+      link="finger3_link3" />
     <axis
       xyz="-0 1 -0" />
@@ -795,5 +793,5 @@
   </joint>
   <link
-    name="finger2_link3">
+    name="finger3_link4">
     <inertial>
       <origin
@@ -835,5 +833,5 @@
   </link>
   <joint
-    name="finger2_joint3"
+    name="finger3_joint4"
     type="revolute">
     <origin
@@ -841,7 +839,7 @@
       rpy="0 0 0" />
     <parent
-      link="finger2_link2" />
-    <child
-      link="finger2_link3" />
+      link="finger3_link3" />
+    <child
+      link="finger3_link4" />
     <axis
       xyz="-0 1 -0" />
@@ -853,5 +851,5 @@
   </joint>
   <link
-    name="finger2_tip_link">
+    name="finger3_tip_link">
     <inertial>
       <origin
@@ -893,5 +891,5 @@
   </link>
   <joint
-    name="finger2_tip_fixed"
+    name="finger3_tip_fixed"
     type="fixed">
     <origin
@@ -899,12 +897,12 @@
       rpy="0 0 0" />
     <parent
-      link="finger2_link3" />
-    <child
-      link="finger2_tip_link" />
+      link="finger3_link4" />
+    <child
+      link="finger3_tip_link" />
     <axis
       xyz="0 0 0" />
   </joint>
   <link
-    name="finger3_link0">
+    name="finger4_link1">
     <inertial>
       <origin
@@ -946,5 +944,5 @@
   </link>
   <joint
-    name="finger3_joint0"
+    name="finger4_joint1"
     type="revolute">
     <origin
@@ -954,5 +952,5 @@
       link="palm_link" />
     <child
-      link="finger3_link0" />
+      link="finger4_link1" />
     <axis
       xyz="-0 1 -0" />
@@ -964,5 +962,5 @@
   </joint>
   <link
-    name="finger3_link1">
+    name="finger4_link2">
     <inertial>
       <origin
@@ -1004,5 +1002,5 @@
   </link>
   <joint
-    name="finger3_joint1"
+    name="finger4_joint2"
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