Commit message: Add OmniPicker to the marvin system, using the previously completed SDK. Notice that I didn't add a URDF visualization of the omnipicker.

File: ros2_control_marvin/description/ros2_control/marvin_dual_system.ros2_control.xacro (robot description, xacro)
@@ -1,5 +1,8 @@
 <?xml version="1.0"?>
 <robot xmlns:xacro="http://www.ros.org/wiki/xacro">
-  <xacro:macro name="marvin_dual_ros2_control" params="name">
+  <xacro:macro name="marvin_dual_ros2_control"
+               params="name
+                       use_gripper_L:=false  gripper_L_arm:=A  gripper_L_can_id:=1
+                       use_gripper_R:=false  gripper_R_arm:=B  gripper_R_can_id:=2">
     <ros2_control name="${name}" type="system">
       <hardware>
@@ -127,4 +130,30 @@
         <state_interface name="velocity"/>
       </joint>
+      <!-- Optional: OmniPicker gripper on left arm -->
+      <xacro:if value="${str(use_gripper_L).lower() == 'true'}">
+        <joint name="gripper_L">
+          <param name="type">omnipicker</param>
+          <param name="arm_side">${gripper_L_arm}</param>
+          <param name="can_node_id">${gripper_L_can_id}</param>
+          <command_interface name="position">
+            <param name="min">0.0</param>
+            <param name="max">1.0</param>
+          </command_interface>
+          <state_interface name="position"/>
+        </joint>
+      </xacro:if>
+      <!-- Optional: OmniPicker gripper on right arm -->
+      <xacro:if value="${str(use_gripper_R).lower() == 'true'}">
+        <joint name="gripper_R">
+          <param name="type">omnipicker</param>
+          <param name="arm_side">${gripper_R_arm}</param>
+          <param name="can_node_id">${gripper_R_can_id}</param>
+          <command_interface name="position">
+            <param name="min">0.0</param>
+            <param name="max">1.0</param>
+          </command_interface>
+          <state_interface name="position"/>
+        </joint>
+      </xacro:if>
     </ros2_control>
   </xacro:macro>
