Commit message: Massive changes.

File: marvin_system/description/ros2_control/marvin_dual_system.ros2_control.xacro (robot description, xacro)
@@ -4,5 +4,14 @@
                params="name
                        use_mock_hardware:=false
-                       joint_vel_ratio:=80  joint_acc_ratio:=80
+                       joint_vel_ratio:=100  joint_acc_ratio:=100
+                       joint_impedance_enabled:=true
+                       joint_impedance_k_left:='2 2 2 2 2 1 1'
+                       joint_impedance_d_left:='0.4 0.4 0.4 0.4 0.4 0.4 0.4'
+                       joint_impedance_k_right:='2 2 2 2 2 1 1'
+                       joint_impedance_d_right:='0.4 0.4 0.4 0.4 0.4 0.4 0.4'
+                       tool_kine_left:='0 0 0 0 0 0'
+                       tool_dyn_left:='0 0 0 0 0 0 0 0 0 0'
+                       tool_kine_right:='0 0 0 0 0 0'
+                       tool_dyn_right:='0 0 0 0 0 0 0 0 0 0'
                        gripper_velocity:=255  gripper_acceleration:=255
                        gripper_command_rate_hz:=50.0  gripper_command_epsilon:=0.001
@@ -30,4 +39,13 @@
           <param name="joint_vel_ratio">${joint_vel_ratio}</param>
           <param name="joint_acc_ratio">${joint_acc_ratio}</param>
+          <param name="joint_impedance_enabled">${joint_impedance_enabled}</param>
+          <param name="joint_impedance_k_left">${joint_impedance_k_left}</param>
+          <param name="joint_impedance_d_left">${joint_impedance_d_left}</param>
+          <param name="joint_impedance_k_right">${joint_impedance_k_right}</param>
+          <param name="joint_impedance_d_right">${joint_impedance_d_right}</param>
+          <param name="tool_kine_left">${tool_kine_left}</param>
+          <param name="tool_dyn_left">${tool_dyn_left}</param>
+          <param name="tool_kine_right">${tool_kine_right}</param>
+          <param name="tool_dyn_right">${tool_dyn_right}</param>
           <param name="gripper_velocity">${gripper_velocity}</param>
           <param name="gripper_acceleration">${gripper_acceleration}</param>
@@ -37,4 +55,8 @@
           <param name="connect_timeout_ms">1500</param>
           <param name="state_timeout_ms">8000</param>
+          <param name="profile_switch_timeout_ms">5000</param>
+          <param name="profile_switch_post_monitor_ms">500</param>
+          <param name="profile_switch_initial_resend_delay_ms">80</param>
+          <param name="profile_switch_resend_interval_ms">20</param>
           <param name="activation_retry_settle_ms">2000</param>
           <param name="activation_max_attempts">3</param>
@@ -80,4 +102,12 @@
         <state_interface name="position"/>
         <state_interface name="velocity"/>
+        <state_interface name="sdk_command_position"/>
+        <state_interface name="active_control_profile"/>
+        <state_interface name="requested_control_profile"/>
+        <state_interface name="sdk_cur_state"/>
+        <state_interface name="sdk_cmd_state"/>
+        <state_interface name="sdk_err_code"/>
+        <state_interface name="sdk_in_frame_serial"/>
+        <state_interface name="sdk_out_frame_serial"/>
       </joint>
       <joint name="Joint2_L">
@@ -89,4 +119,5 @@
         <state_interface name="position"/>
         <state_interface name="velocity"/>
+        <state_interface name="sdk_command_position"/>
       </joint>
       <joint name="Joint3_L">
@@ -98,4 +129,5 @@
         <state_interface name="position"/>
         <state_interface name="velocity"/>
+        <state_interface name="sdk_command_position"/>
       </joint>
       <joint name="Joint4_L">
@@ -107,4 +139,5 @@
         <state_interface name="position"/>
         <state_interface name="velocity"/>
+        <state_interface name="sdk_command_position"/>
       </joint>
       <joint name="Joint5_L">
@@ -116,4 +149,5 @@
         <state_interface name="position"/>
         <state_interface name="velocity"/>
+        <state_interface name="sdk_command_position"/>
       </joint>
       <joint name="Joint6_L">
@@ -125,4 +159,5 @@
         <state_interface name="position"/>
         <state_interface name="velocity"/>
+        <state_interface name="sdk_command_position"/>
       </joint>
       <joint name="Joint7_L">
@@ -134,4 +169,5 @@
         <state_interface name="position"/>
         <state_interface name="velocity"/>
+        <state_interface name="sdk_command_position"/>
       </joint>
       <!-- Right arm (SDK arm B, index 1) — joints 7..13 -->
@@ -144,4 +180,10 @@
         <state_interface name="position"/>
         <state_interface name="velocity"/>
+        <state_interface name="sdk_command_position"/>
+        <state_interface name="sdk_cur_state"/>
+        <state_interface name="sdk_cmd_state"/>
+        <state_interface name="sdk_err_code"/>
+        <state_interface name="sdk_in_frame_serial"/>
+        <state_interface name="sdk_out_frame_serial"/>
       </joint>
       <joint name="Joint2_R">
@@ -153,4 +195,5 @@
         <state_interface name="position"/>
         <state_interface name="velocity"/>
+        <state_interface name="sdk_command_position"/>
       </joint>
       <joint name="Joint3_R">
@@ -162,4 +205,5 @@
         <state_interface name="position"/>
         <state_interface name="velocity"/>
+        <state_interface name="sdk_command_position"/>
       </joint>
       <joint name="Joint4_R">
@@ -171,4 +215,5 @@
         <state_interface name="position"/>
         <state_interface name="velocity"/>
+        <state_interface name="sdk_command_position"/>
       </joint>
       <joint name="Joint5_R">
@@ -180,4 +225,5 @@
         <state_interface name="position"/>
         <state_interface name="velocity"/>
+        <state_interface name="sdk_command_position"/>
       </joint>
       <joint name="Joint6_R">
@@ -189,4 +235,5 @@
         <state_interface name="position"/>
         <state_interface name="velocity"/>
+        <state_interface name="sdk_command_position"/>
       </joint>
       <joint name="Joint7_R">
@@ -198,4 +245,5 @@
         <state_interface name="position"/>
         <state_interface name="velocity"/>
+        <state_interface name="sdk_command_position"/>
       </joint>
       <!-- Optional: OmniPicker gripper on left arm -->

File: wujihand_system/description/ros2_control/wujihand-right.ros2_control.xacro (robot description, xacro)
@@ -1,180 +1,200 @@
 <?xml version="1.0"?>
 <robot xmlns:xacro="http://www.ros.org/wiki/xacro">
-	<!--
-		Usage (example):
-			<xacro:include filename="$(find-pkg-share wujihand_system)/description/ros2_control/wujihand-right.ros2_control.xacro"/>
-			<xacro:wujihand_right_ros2_control name="wujihand_right"/>
-	-->
-	<xacro:macro name="wujihand_right_ros2_control" params="name">
-		<ros2_control name="${name}" type="system">
-			<hardware>
-				<plugin>wujihand_system/WujiHandHardware</plugin>
-                <param name="low_pass_cutoff_frequency">5.0</param>
-			</hardware>
-			<!--
-				Joint limits from provided table:
-					Finger 0..4 Joint 0..3  ->  finger0..4_joint0..3
-			-->
-			<joint name="finger0_joint0">
-				<command_interface name="position">
-					<param name="min">-0.0343273</param>
-					<param name="max">1.74405</param>
-				</command_interface>
-				<state_interface name="position"/>
-				<state_interface name="velocity"/>
-			</joint>
-			<joint name="finger0_joint1">
-				<command_interface name="position">
-					<param name="min">-0.241261</param>
-					<param name="max">0.945935</param>
-				</command_interface>
-				<state_interface name="position"/>
-				<state_interface name="velocity"/>
-			</joint>
-			<joint name="finger0_joint2">
-				<command_interface name="position">
-					<param name="min">-0.540319</param>
-					<param name="max">1.7011</param>
-				</command_interface>
-				<state_interface name="position"/>
-				<state_interface name="velocity"/>
-			</joint>
-			<joint name="finger0_joint3">
-				<command_interface name="position">
-					<param name="min">-0.584444</param>
-					<param name="max">1.63935</param>
-				</command_interface>
-				<state_interface name="position"/>
-				<state_interface name="velocity"/>
-			</joint>
-			<joint name="finger1_joint0">
-				<command_interface name="position">
-					<param name="min">-0.283902</param>
-					<param name="max">1.62698</param>
-				</command_interface>
-				<state_interface name="position"/>
-				<state_interface name="velocity"/>
-			</joint>
-			<joint name="finger1_joint1">
-				<command_interface name="position">
-					<param name="min">-0.540946</param>
-					<param name="max">0.448065</param>
-				</command_interface>
-				<state_interface name="position"/>
-				<state_interface name="velocity"/>
-			</joint>
-			<joint name="finger1_joint2">
-				<command_interface name="position">
-					<param name="min">-0.551836</param>
-					<param name="max">1.66596</param>
-				</command_interface>
-				<state_interface name="position"/>
-				<state_interface name="velocity"/>
-			</joint>
-			<joint name="finger1_joint3">
-				<command_interface name="position">
-					<param name="min">-0.568183</param>
-					<param name="max">1.69382</param>
-				</command_interface>
-				<state_interface name="position"/>
-				<state_interface name="velocity"/>
-			</joint>
-			<joint name="finger2_joint0">
-				<command_interface name="position">
-					<param name="min">-0.274021</param>
-					<param name="max">1.63671</param>
-				</command_interface>
-				<state_interface name="position"/>
-				<state_interface name="velocity"/>
-			</joint>
-			<joint name="finger2_joint1">
-				<command_interface name="position">
-					<param name="min">-0.45005</param>
-					<param name="max">0.339799</param>
-				</command_interface>
-				<state_interface name="position"/>
-				<state_interface name="velocity"/>
-			</joint>
-			<joint name="finger2_joint2">
-				<command_interface name="position">
-					<param name="min">-0.58411</param>
-					<param name="max">1.63868</param>
-				</command_interface>
-				<state_interface name="position"/>
-				<state_interface name="velocity"/>
-			</joint>
-			<joint name="finger2_joint3">
-				<command_interface name="position">
-					<param name="min">-0.545375</param>
-					<param name="max">1.72185</param>
-				</command_interface>
-				<state_interface name="position"/>
-				<state_interface name="velocity"/>
-			</joint>
-			<joint name="finger3_joint0">
-				<command_interface name="position">
-					<param name="min">-0.248642</param>
-					<param name="max">1.65442</param>
-				</command_interface>
-				<state_interface name="position"/>
-				<state_interface name="velocity"/>
-			</joint>
-			<joint name="finger3_joint1">
-				<command_interface name="position">
-					<param name="min">-0.418249</param>
-					<param name="max">0.369714</param>
-				</command_interface>
-				<state_interface name="position"/>
-				<state_interface name="velocity"/>
-			</joint>
-			<joint name="finger3_joint2">
-				<command_interface name="position">
-					<param name="min">-0.571115</param>
-					<param name="max">1.65579</param>
-				</command_interface>
-				<state_interface name="position"/>
-				<state_interface name="velocity"/>
-			</joint>
-			<joint name="finger3_joint3">
-				<command_interface name="position">
-					<param name="min">-0.566777</param>
-					<param name="max">1.69417</param>
-				</command_interface>
-				<state_interface name="position"/>
-				<state_interface name="velocity"/>
-			</joint>
-			<joint name="finger4_joint0">
-				<command_interface name="position">
-					<param name="min">-0.25879</param>
-					<param name="max">1.6567</param>
-				</command_interface>
-				<state_interface name="position"/>
-				<state_interface name="velocity"/>
-			</joint>
-			<joint name="finger4_joint1">
-				<command_interface name="position">
-					<param name="min">-0.412827</param>
-					<param name="max">0.396453</param>
-				</command_interface>
-				<state_interface name="position"/>
-				<state_interface name="velocity"/>
-			</joint>
-			<joint name="finger4_joint2">
-				<command_interface name="position">
-					<param name="min">-0.556739</param>
-					<param name="max">1.68019</param>
-				</command_interface>
-				<state_interface name="position"/>
-				<state_interface name="velocity"/>
-			</joint>
-			<joint name="finger4_joint3">
-				<command_interface name="position">
-					<param name="min">-0.572835</param>
-					<param name="max">1.69304</param>
-				</command_interface>
-				<state_interface name="position"/>
-				<state_interface name="velocity"/>
-			</joint>
-		</ros2_control>
-	</xacro:macro>
+  <xacro:macro name="wujihand_right_ros2_control" params="name use_mock_hardware usb_serial_number expected_handedness">
+    <ros2_control name="${name}" type="system">
+      <hardware>
+        <xacro:if value="${str(use_mock_hardware).lower() == 'true'}">
+          <plugin>mock_components/GenericSystem</plugin>
+          <param name="mock_sensor_commands">false</param>
+          <param name="state_following_offset">0.0</param>
+        </xacro:if>
+        <xacro:unless value="${str(use_mock_hardware).lower() == 'true'}">
+          <plugin>wujihand_system/WujiHandHardware</plugin>
+          <param name="low_pass_cutoff_frequency">5.0</param>
+          <param name="usb_serial_number">${usb_serial_number}</param>
+          <param name="expected_handedness">${expected_handedness}</param>
+        </xacro:unless>
+      </hardware>
+      <joint name="right_finger1_joint1">
+        <command_interface name="position">
+          <param name="min">0.0475</param>
+          <param name="max">1.6033</param>
+          <param name="initial_value">0.0475</param>
+        </command_interface>
+        <state_interface name="position"/>
+        <state_interface name="velocity"/>
+      </joint>
+      <joint name="right_finger1_joint2">
+        <command_interface name="position">
+          <param name="min">-0.1387</param>
+          <param name="max">0.9324</param>
+          <param name="initial_value">0.0</param>
+        </command_interface>
+        <state_interface name="position"/>
+        <state_interface name="velocity"/>
+      </joint>
+      <joint name="right_finger1_joint3">
+        <command_interface name="position">
+          <param name="min">-0.4642</param>
+          <param name="max">1.5623</param>
+          <param name="initial_value">0.0</param>
+        </command_interface>
+        <state_interface name="position"/>
+        <state_interface name="velocity"/>
+      </joint>
+      <joint name="right_finger1_joint4">
+        <command_interface name="position">
+          <param name="min">-0.4699</param>
+          <param name="max">1.5568</param>
+          <param name="initial_value">0.0</param>
+        </command_interface>
+        <state_interface name="position"/>
+        <state_interface name="velocity"/>
+      </joint>
+      <joint name="right_finger2_joint1">
+        <command_interface name="position">
+          <param name="min">-0.1585</param>
+          <param name="max">1.5604</param>
+          <param name="initial_value">0.0</param>
+        </command_interface>
+        <state_interface name="position"/>
+        <state_interface name="velocity"/>
+      </joint>
+      <joint name="right_finger2_joint2">
+        <command_interface name="position">
+          <param name="min">-0.37</param>
+          <param name="max">0.37</param>
+          <param name="initial_value">0.0</param>
+        </command_interface>
+        <state_interface name="position"/>
+        <state_interface name="velocity"/>
+      </joint>
+      <joint name="right_finger2_joint3">
+        <command_interface name="position">
+          <param name="min">-0.4777</param>
+          <param name="max">1.5485</param>
+          <param name="initial_value">0.0</param>
+        </command_interface>
+        <state_interface name="position"/>
+        <state_interface name="velocity"/>
+      </joint>
+      <joint name="right_finger2_joint4">
+        <command_interface name="position">
+          <param name="min">-0.4683</param>
+          <param name="max">1.5753</param>
+          <param name="initial_value">0.0</param>
+        </command_interface>
+        <state_interface name="position"/>
+        <state_interface name="velocity"/>
+      </joint>
+      <joint name="right_finger3_joint1">
+        <command_interface name="position">
+          <param name="min">-0.1644</param>
+          <param name="max">1.5516</param>
+          <param name="initial_value">0.0</param>
+        </command_interface>
+        <state_interface name="position"/>
+        <state_interface name="velocity"/>
+      </joint>
+      <joint name="right_finger3_joint2">
+        <command_interface name="position">
+          <param name="min">-0.37</param>
+          <param name="max">0.37</param>
+          <param name="initial_value">0.0</param>
+        </command_interface>
+        <state_interface name="position"/>
+        <state_interface name="velocity"/>
+      </joint>
+      <joint name="right_finger3_joint3">
+        <command_interface name="position">
+          <param name="min">-0.4739</param>
+          <param name="max">1.5512</param>
+          <param name="initial_value">0.0</param>
+        </command_interface>
+        <state_interface name="position"/>
+        <state_interface name="velocity"/>
+      </joint>
+      <joint name="right_finger3_joint4">
+        <command_interface name="position">
+          <param name="min">-0.4684</param>
+          <param name="max">1.5745</param>
+          <param name="initial_value">0.0</param>
+        </command_interface>
+        <state_interface name="position"/>
+        <state_interface name="velocity"/>
+      </joint>
+      <joint name="right_finger4_joint1">
+        <command_interface name="position">
+          <param name="min">-0.1554</param>
+          <param name="max">1.5585</param>
+          <param name="initial_value">0.0</param>
+        </command_interface>
+        <state_interface name="position"/>
+        <state_interface name="velocity"/>
+      </joint>
+      <joint name="right_finger4_joint2">
+        <command_interface name="position">
+          <param name="min">-0.37</param>
+          <param name="max">0.37</param>
+          <param name="initial_value">0.0</param>
+        </command_interface>
+        <state_interface name="position"/>
+        <state_interface name="velocity"/>
+      </joint>
+      <joint name="right_finger4_joint3">
+        <command_interface name="position">
+          <param name="min">-0.4765</param>
+          <param name="max">1.5487</param>
+          <param name="initial_value">0.0</param>
+        </command_interface>
+        <state_interface name="position"/>
+        <state_interface name="velocity"/>
+      </joint>
+      <joint name="right_finger4_joint4">
+        <command_interface name="position">
+          <param name="min">-0.4777</param>
+          <param name="max">1.5634</param>
+          <param name="initial_value">0.0</param>
+        </command_interface>
+        <state_interface name="position"/>
+        <state_interface name="velocity"/>
+      </joint>
+      <joint name="right_finger5_joint1">
+        <command_interface name="position">
+          <param name="min">-0.1626</param>
+          <param name="max">1.5585</param>
+          <param name="initial_value">0.0</param>
+        </command_interface>
+        <state_interface name="position"/>
+        <state_interface name="velocity"/>
+      </joint>
+      <joint name="right_finger5_joint2">
+        <command_interface name="position">
+          <param name="min">-0.37</param>
+          <param name="max">0.37</param>
+          <param name="initial_value">0.0</param>
+        </command_interface>
+        <state_interface name="position"/>
+        <state_interface name="velocity"/>
+      </joint>
+      <joint name="right_finger5_joint3">
+        <command_interface name="position">
+          <param name="min">-0.4768</param>
+          <param name="max">1.5490</param>
+          <param name="initial_value">0.0</param>
+        </command_interface>
+        <state_interface name="position"/>
+        <state_interface name="velocity"/>
+      </joint>
+      <joint name="right_finger5_joint4">
+        <command_interface name="position">
+          <param name="min">-0.4683</param>
+          <param name="max">1.5735</param>
+          <param name="initial_value">0.0</param>
+        </command_interface>
+        <state_interface name="position"/>
+        <state_interface name="velocity"/>
+      </joint>
+    </ros2_control>
+  </xacro:macro>
 </robot>

File: wujihand_system/description/urdf/wujihand-right.urdf (robot description, URDF)
Before this commit: robot wujihand-right, 0 links, 0 joints
Links:
- added link world
Joints:
- added joint world_to_right_palm: type fixed, parent world, child right_palm_link, origin xyz=$(arg mount_xyz) rpy=$(arg mount_rpy)
