Commit message: The hand posture is generally correct, but there is a problem with the urdf.

File: wujihand_system/description/ros2_control/wujihand-left.ros2_control.xacro (robot description, xacro)
@@ -18,7 +18,7 @@
       <joint name="left_finger1_joint1">
         <command_interface name="position">
-          <param name="min">0.0475</param>
-          <param name="max">1.6033</param>
-          <param name="initial_value">0.0475</param>
+          <param name="min">0.0583</param>
+          <param name="max">1.5941</param>
+          <param name="initial_value">0.0583</param>
         </command_interface>
         <state_interface name="position"/>
@@ -27,6 +27,6 @@
       <joint name="left_finger1_joint2">
         <command_interface name="position">
-          <param name="min">-0.1387</param>
-          <param name="max">0.9324</param>
+          <param name="min">-0.1199</param>
+          <param name="max">0.9335</param>
           <param name="initial_value">0.0</param>
         </command_interface>
@@ -36,6 +36,6 @@
       <joint name="left_finger1_joint3">
         <command_interface name="position">
-          <param name="min">-0.4642</param>
-          <param name="max">1.5623</param>
+          <param name="min">-0.4646</param>
+          <param name="max">1.5639</param>
           <param name="initial_value">0.0</param>
         </command_interface>
@@ -45,6 +45,6 @@
       <joint name="left_finger1_joint4">
         <command_interface name="position">
-          <param name="min">-0.4699</param>
-          <param name="max">1.5568</param>
+          <param name="min">-0.4570</param>
+          <param name="max">1.5684</param>
           <param name="initial_value">0.0</param>
         </command_interface>
@@ -54,6 +54,6 @@
       <joint name="left_finger2_joint1">
         <command_interface name="position">
-          <param name="min">-0.1585</param>
-          <param name="max">1.5604</param>
+          <param name="min">-0.1560</param>
+          <param name="max">1.5619</param>
           <param name="initial_value">0.0</param>
         </command_interface>
@@ -63,6 +63,6 @@
       <joint name="left_finger2_joint2">
         <command_interface name="position">
-          <param name="min">-0.37</param>
-          <param name="max">0.37</param>
+          <param name="min">-0.4095</param>
+          <param name="max">0.2921</param>
           <param name="initial_value">0.0</param>
         </command_interface>
@@ -72,6 +72,6 @@
       <joint name="left_finger2_joint3">
         <command_interface name="position">
-          <param name="min">-0.4777</param>
-          <param name="max">1.5485</param>
+          <param name="min">-0.4839</param>
+          <param name="max">1.5466</param>
           <param name="initial_value">0.0</param>
         </command_interface>
@@ -81,6 +81,6 @@
       <joint name="left_finger2_joint4">
         <command_interface name="position">
-          <param name="min">-0.4683</param>
-          <param name="max">1.5753</param>
+          <param name="min">-0.4723</param>
+          <param name="max">1.5754</param>
           <param name="initial_value">0.0</param>
         </command_interface>
@@ -90,6 +90,6 @@
       <joint name="left_finger3_joint1">
         <command_interface name="position">
-          <param name="min">-0.1644</param>
-          <param name="max">1.5516</param>
+          <param name="min">-0.1569</param>
+          <param name="max">1.5536</param>
           <param name="initial_value">0.0</param>
         </command_interface>
@@ -99,6 +99,6 @@
       <joint name="left_finger3_joint2">
         <command_interface name="position">
-          <param name="min">-0.37</param>
-          <param name="max">0.37</param>
+          <param name="min">-0.3977</param>
+          <param name="max">0.3115</param>
           <param name="initial_value">0.0</param>
         </command_interface>
@@ -108,6 +108,6 @@
       <joint name="left_finger3_joint3">
         <command_interface name="position">
-          <param name="min">-0.4739</param>
-          <param name="max">1.5512</param>
+          <param name="min">-0.4847</param>
+          <param name="max">1.5411</param>
           <param name="initial_value">0.0</param>
         </command_interface>
@@ -117,6 +117,6 @@
       <joint name="left_finger3_joint4">
         <command_interface name="position">
-          <param name="min">-0.4684</param>
-          <param name="max">1.5745</param>
+          <param name="min">-0.4671</param>
+          <param name="max">1.5788</param>
           <param name="initial_value">0.0</param>
         </command_interface>
@@ -126,6 +126,6 @@
       <joint name="left_finger4_joint1">
         <command_interface name="position">
-          <param name="min">-0.1554</param>
-          <param name="max">1.5585</param>
+          <param name="min">-0.1507</param>
+          <param name="max">1.5636</param>
           <param name="initial_value">0.0</param>
         </command_interface>
@@ -135,6 +135,6 @@
       <joint name="left_finger4_joint2">
         <command_interface name="position">
-          <param name="min">-0.37</param>
-          <param name="max">0.37</param>
+          <param name="min">-0.4101</param>
+          <param name="max">0.3014</param>
           <param name="initial_value">0.0</param>
         </command_interface>
@@ -144,6 +144,6 @@
       <joint name="left_finger4_joint3">
         <command_interface name="position">
-          <param name="min">-0.4765</param>
-          <param name="max">1.5487</param>
+          <param name="min">-0.4747</param>
+          <param name="max">1.5526</param>
           <param name="initial_value">0.0</param>
         </command_interface>
@@ -153,6 +153,6 @@
       <joint name="left_finger4_joint4">
         <command_interface name="position">
-          <param name="min">-0.4777</param>
-          <param name="max">1.5634</param>
+          <param name="min">-0.4729</param>
+          <param name="max">1.5718</param>
           <param name="initial_value">0.0</param>
         </command_interface>
@@ -162,6 +162,6 @@
       <joint name="left_finger5_joint1">
         <command_interface name="position">
-          <param name="min">-0.1626</param>
-          <param name="max">1.5585</param>
+          <param name="min">-0.1578</param>
+          <param name="max">1.5632</param>
           <param name="initial_value">0.0</param>
         </command_interface>
@@ -171,6 +171,6 @@
       <joint name="left_finger5_joint2">
         <command_interface name="position">
-          <param name="min">-0.37</param>
-          <param name="max">0.37</param>
+          <param name="min">-0.4103</param>
+          <param name="max">0.2949</param>
           <param name="initial_value">0.0</param>
         </command_interface>
@@ -180,6 +180,6 @@
       <joint name="left_finger5_joint3">
         <command_interface name="position">
-          <param name="min">-0.4768</param>
-          <param name="max">1.5490</param>
+          <param name="min">-0.4733</param>
+          <param name="max">1.5560</param>
           <param name="initial_value">0.0</param>
         </command_interface>
@@ -189,6 +189,6 @@
       <joint name="left_finger5_joint4">
         <command_interface name="position">
-          <param name="min">-0.4683</param>
-          <param name="max">1.5735</param>
+          <param name="min">-0.4662</param>
+          <param name="max">1.5760</param>
           <param name="initial_value">0.0</param>
         </command_interface>

File: wujihand_system/description/ros2_control/wujihand-right.ros2_control.xacro (robot description, xacro)
@@ -18,7 +18,7 @@
       <joint name="right_finger1_joint1">
         <command_interface name="position">
-          <param name="min">0.0475</param>
-          <param name="max">1.6033</param>
-          <param name="initial_value">0.0475</param>
+          <param name="min">0.0368</param>
+          <param name="max">1.6125</param>
+          <param name="initial_value">0.0368</param>
         </command_interface>
         <state_interface name="position"/>
@@ -27,6 +27,6 @@
       <joint name="right_finger1_joint2">
         <command_interface name="position">
-          <param name="min">-0.1387</param>
-          <param name="max">0.9324</param>
+          <param name="min">-0.1576</param>
+          <param name="max">0.9312</param>
           <param name="initial_value">0.0</param>
         </command_interface>
@@ -36,6 +36,6 @@
       <joint name="right_finger1_joint3">
         <command_interface name="position">
-          <param name="min">-0.4642</param>
-          <param name="max">1.5623</param>
+          <param name="min">-0.4638</param>
+          <param name="max">1.5607</param>
           <param name="initial_value">0.0</param>
         </command_interface>
@@ -45,6 +45,6 @@
       <joint name="right_finger1_joint4">
         <command_interface name="position">
-          <param name="min">-0.4699</param>
-          <param name="max">1.5568</param>
+          <param name="min">-0.4829</param>
+          <param name="max">1.5451</param>
           <param name="initial_value">0.0</param>
         </command_interface>
@@ -54,6 +54,6 @@
       <joint name="right_finger2_joint1">
         <command_interface name="position">
-          <param name="min">-0.1585</param>
-          <param name="max">1.5604</param>
+          <param name="min">-0.1611</param>
+          <param name="max">1.5588</param>
           <param name="initial_value">0.0</param>
         </command_interface>
@@ -63,6 +63,6 @@
       <joint name="right_finger2_joint2">
         <command_interface name="position">
-          <param name="min">-0.37</param>
-          <param name="max">0.37</param>
+          <param name="min">-0.4044</param>
+          <param name="max">0.3054</param>
           <param name="initial_value">0.0</param>
         </command_interface>
@@ -72,6 +72,6 @@
       <joint name="right_finger2_joint3">
         <command_interface name="position">
-          <param name="min">-0.4777</param>
-          <param name="max">1.5485</param>
+          <param name="min">-0.4714</param>
+          <param name="max">1.5504</param>
           <param name="initial_value">0.0</param>
         </command_interface>
@@ -81,5 +81,5 @@
       <joint name="right_finger2_joint4">
         <command_interface name="position">
-          <param name="min">-0.4683</param>
+          <param name="min">-0.4644</param>
           <param name="max">1.5753</param>
           <param name="initial_value">0.0</param>
@@ -90,6 +90,6 @@
       <joint name="right_finger3_joint1">
         <command_interface name="position">
-          <param name="min">-0.1644</param>
-          <param name="max">1.5516</param>
+          <param name="min">-0.1719</param>
+          <param name="max">1.5496</param>
           <param name="initial_value">0.0</param>
         </command_interface>
@@ -99,6 +99,6 @@
       <joint name="right_finger3_joint2">
         <command_interface name="position">
-          <param name="min">-0.37</param>
-          <param name="max">0.37</param>
+          <param name="min">-0.4014</param>
+          <param name="max">0.2996</param>
           <param name="initial_value">0.0</param>
         </command_interface>
@@ -108,6 +108,6 @@
       <joint name="right_finger3_joint3">
         <command_interface name="position">
-          <param name="min">-0.4739</param>
-          <param name="max">1.5512</param>
+          <param name="min">-0.4632</param>
+          <param name="max">1.5613</param>
           <param name="initial_value">0.0</param>
         </command_interface>
@@ -117,6 +117,6 @@
       <joint name="right_finger3_joint4">
         <command_interface name="position">
-          <param name="min">-0.4684</param>
-          <param name="max">1.5745</param>
+          <param name="min">-0.4697</param>
+          <param name="max">1.5702</param>
           <param name="initial_value">0.0</param>
         </command_interface>
@@ -126,6 +126,6 @@
       <joint name="right_finger4_joint1">
         <command_interface name="position">
-          <param name="min">-0.1554</param>
-          <param name="max">1.5585</param>
+          <param name="min">-0.1601</param>
+          <param name="max">1.5534</param>
           <param name="initial_value">0.0</param>
         </command_interface>
@@ -135,6 +135,6 @@
       <joint name="right_finger4_joint2">
         <command_interface name="position">
-          <param name="min">-0.37</param>
-          <param name="max">0.37</param>
+          <param name="min">-0.4134</param>
+          <param name="max">0.3161</param>
           <param name="initial_value">0.0</param>
         </command_interface>
@@ -144,6 +144,6 @@
       <joint name="right_finger4_joint3">
         <command_interface name="position">
-          <param name="min">-0.4765</param>
-          <param name="max">1.5487</param>
+          <param name="min">-0.4782</param>
+          <param name="max">1.5448</param>
           <param name="initial_value">0.0</param>
         </command_interface>
@@ -153,6 +153,6 @@
       <joint name="right_finger4_joint4">
         <command_interface name="position">
-          <param name="min">-0.4777</param>
-          <param name="max">1.5634</param>
+          <param name="min">-0.4825</param>
+          <param name="max">1.5550</param>
           <param name="initial_value">0.0</param>
         </command_interface>
@@ -162,6 +162,6 @@
       <joint name="right_finger5_joint1">
         <command_interface name="position">
-          <param name="min">-0.1626</param>
-          <param name="max">1.5585</param>
+          <param name="min">-0.1674</param>
+          <param name="max">1.5539</param>
           <param name="initial_value">0.0</param>
         </command_interface>
@@ -171,6 +171,6 @@
       <joint name="right_finger5_joint2">
         <command_interface name="position">
-          <param name="min">-0.37</param>
-          <param name="max">0.37</param>
+          <param name="min">-0.4203</param>
+          <param name="max">0.2931</param>
           <param name="initial_value">0.0</param>
         </command_interface>
@@ -180,6 +180,6 @@
       <joint name="right_finger5_joint3">
         <command_interface name="position">
-          <param name="min">-0.4768</param>
-          <param name="max">1.5490</param>
+          <param name="min">-0.4804</param>
+          <param name="max">1.5420</param>
           <param name="initial_value">0.0</param>
         </command_interface>
@@ -189,6 +189,6 @@
       <joint name="right_finger5_joint4">
         <command_interface name="position">
-          <param name="min">-0.4683</param>
-          <param name="max">1.5735</param>
+          <param name="min">-0.4705</param>
+          <param name="max">1.5709</param>
           <param name="initial_value">0.0</param>
         </command_interface>
