Commit message: The hand posture is generally correct, but there is a problem with the urdf.

File: wujihand_system/third_party/wuji_retargeting/wuji_retargeting/wuji_hand_description/urdf/left.urdf (robot description, URDF)
Before this commit: robot wujihand-left-v1.0.2, 26 links, 25 joints
Links:
- link finger1_link1: geometry collision mesh filename=finger1_link1.STL; visual mesh filename=finger1_link1.STL
- link finger1_link2: geometry collision mesh filename=finger1_link2.STL; visual mesh filename=finger1_link2.STL
- link finger1_link3: geometry collision mesh filename=finger1_link3.STL; visual mesh filename=finger1_link3.STL
- link finger1_link4: geometry collision mesh filename=finger1_link4.STL; visual mesh filename=finger1_link4.STL
- link finger1_tip_link: mass 0.004 -> 0.0041; geometry collision mesh filename=finger1_tip_link.STL; visual mesh filename=finger1_tip_link.STL
- link finger2_link1: geometry collision mesh filename=finger2_link1.STL; visual mesh filename=finger2_link1.STL
- link finger2_link2: geometry collision mesh filename=finger2_link2.STL; visual mesh filename=finger2_link2.STL
- link finger2_link3: geometry collision mesh filename=finger2_link3.STL; visual mesh filename=finger2_link3.STL
- link finger2_link4: geometry collision mesh filename=finger2_link4.STL; visual mesh filename=finger2_link4.STL
- link finger2_tip_link: mass 0.004 -> 0.00318; geometry collision mesh filename=finger2_tip_link.STL; visual mesh filename=finger2_tip_link.STL
- link finger3_link1: geometry collision mesh filename=finger3_link1.STL; visual mesh filename=finger3_link1.STL
- link finger3_link2: geometry collision mesh filename=finger3_link2.STL; visual mesh filename=finger3_link2.STL
- link finger3_link3: geometry collision mesh filename=finger3_link3.STL; visual mesh filename=finger3_link3.STL
- link finger3_link4: geometry collision mesh filename=finger3_link4.STL; visual mesh filename=finger3_link4.STL
- link finger3_tip_link: mass 0.004 -> 0.00318; geometry collision mesh filename=finger3_tip_link.STL; visual mesh filename=finger3_tip_link.STL
- link finger4_link1: geometry collision mesh filename=finger4_link1.STL; visual mesh filename=finger4_link1.STL
- link finger4_link2: geometry collision mesh filename=finger4_link2.STL; visual mesh filename=finger4_link2.STL
- link finger4_link3: geometry collision mesh filename=finger4_link3.STL; visual mesh filename=finger4_link3.STL
- link finger4_link4: geometry collision mesh filename=finger4_link4.STL; visual mesh filename=finger4_link4.STL
- link finger4_tip_link: mass 0.004 -> 0.00318; geometry collision mesh filename=finger4_tip_link.STL; visual mesh filename=finger4_tip_link.STL
- link finger5_link1: geometry collision mesh filename=finger5_link1.STL; visual mesh filename=finger5_link1.STL
- link finger5_link2: geometry collision mesh filename=finger5_link2.STL; visual mesh filename=finger5_link2.STL
- link finger5_link3: geometry collision mesh filename=finger5_link3.STL; visual mesh filename=finger5_link3.STL
- link finger5_link4: geometry collision mesh filename=finger5_link4.STL; visual mesh filename=finger5_link4.STL
- link finger5_tip_link: mass 0.004 -> 0.00318; geometry collision mesh filename=finger5_tip_link.STL; visual mesh filename=finger5_tip_link.STL
- link palm_link: mass 0.2179 -> 0.16914; geometry collision mesh filename=palm_link.STL; visual mesh filename=palm_link.STL
Joints:
- joint finger1_joint1: axis 0 0 1 -> 0 1 0; limit lower=-0.0448 upper=1.6508 effort=0.6 velocity=8.587 -> lower=0.0583 upper=1.5941 effort=0.4452 velocity=8.587; origin xyz=0.0085244 -0.020575 0.028712 rpy=0.38179 -0.2259 -0.92978 -> xyz=0.00843985365597852 -0.0205866432293554 0.0288928344107784 rpy=1.5023139401368 0.43577167910554 3.11264835810693
- joint finger1_joint2: axis 0 0 -1 -> 0 -1 0; limit lower=-0.1659 upper=0.9339 effort=0.6 velocity=11.1 -> lower=-0.1199 upper=0.9335 effort=0.4259 velocity=11.1; origin xyz=0.014132 -0.0047549 0.0060191 rpy=-1.6442 -0.32223 -0.53456 -> xyz=-0.0054483 0.0058191 -0.01388 rpy=0.14937 -0.34623 1.5901
- joint finger1_joint3: axis 0 0 1 -> 0 1 0; limit lower=-0.4932 upper=1.6272 effort=0.3 velocity=12.863 -> lower=-0.4646 upper=1.5639 effort=0.1888 velocity=13.578; origin xyz=0.034664 0.00018873 0.0009916 rpy=1.909 -6.6317E-05 -0.052012 -> xyz=-0.000846961087777298 0.000991504133990267 -0.0346562987377679 rpy=0.0332538563601251 0.0117623260174173 -1.90877003040037
- joint finger1_joint4: axis 0 0 1 -> 0 1 0; limit lower=-0.4932 upper=1.6272 effort=0.3 velocity=13.579 -> lower=-0.4570 upper=1.5684 effort=0.1468 velocity=12.863; origin xyz=0.0295 0 0.00025125 rpy=0 0 0 -> xyz=0 0 -0.0294999998969489 rpy=0 0 0
- joint finger1_tip_fixed: origin xyz=0.0283 -0.0010446 -0.00024656 rpy=0 0 0 -> xyz=0.00104999999999626 0 -0.0235000000000007 rpy=3.14159265358971 0 -3.14159265358979
- joint finger2_joint1: axis 1 0 0 -> 0 1 0; limit lower=-0.32695 upper=1.636 effort=1 velocity=8.203 -> lower=-0.1560 upper=1.5619 effort=0.6188 velocity=8.203; origin xyz=-0.0058701 -0.029434 0.091917 rpy=-0.071558 -0.11043 1.7969 -> xyz=-0.00587008921400943 -0.0294338632807759 0.0919165306703557 rpy=0.110463316505378 -0.0251937198594477 0.223332069867641
- joint finger2_joint2: axis 0 0 -1 -> -1 0 0; limit lower=-0.495 upper=0.495 effort=0.2 velocity=8.1158 -> lower=-0.4095 upper=0.2921 effort=0.1822 velocity=8.115; origin xyz=0 -0.0022 0.004 rpy=1.5708 -1.5708 0 -> xyz=0.000389540189408399 0 0.00402230398376657 rpy=0 -0.0462278050739338 0
- joint finger2_joint3: axis 0 0 1 -> 0 1 0; limit lower=-0.4932 upper=1.6272 effort=0.3 velocity=12.863 -> lower=-0.4839 upper=1.5466 effort=0.2251 velocity=13.578; origin xyz=0.043618 0 -0.00475 rpy=1.5705 0 0 -> xyz=-0.00312502624735005 0.000100282455430194 0.0436176874512652 rpy=0 0 0.000268612717770449
- joint finger2_joint4: axis 0 0 1 -> 0 1 0; limit lower=-0.4932 upper=1.6272 effort=0.3 velocity=13.579 -> lower=-0.4723 upper=1.5754 effort=0.2170 velocity=12.863; origin xyz=0.0295 0 0 rpy=0 0 0 -> xyz=0 0 0.0294999999999921 rpy=0 0 0
- joint finger2_tip_fixed: origin xyz=0.0267 -0.00105 0 rpy=0 0 0 -> xyz=-0.00199999998882132 -9.99999775618474E-05 0.0239466139626726 rpy=0 0 0
- joint finger3_joint1: axis 1 0 0 -> 0 1 0; limit lower=-0.32695 upper=1.63595 effort=1 velocity=8.203 -> lower=-0.1569 upper=1.5536 effort=0.6494 velocity=8.203; origin xyz=-0.01046 -0.0074615 0.089544 rpy=-0.087266 -5.0693E-05 1.5702 -> xyz=-0.01046 -0.0074615 0.089544 rpy=5.0693E-05 0 -0.00057944
- joint finger3_joint2: axis 0 0 -1 -> -1 0 0; limit lower=-0.495 upper=0.495 effort=0.2 velocity=8.115 -> lower=-0.3977 upper=0.3115 effort=0.1827 velocity=8.115; origin xyz=0 -0.0022 0.004 rpy=1.5708 -1.5708 0 -> xyz=0.000224188923157675 0 0.00403489896760838 rpy=0 -0.0872664630099629 0
- joint finger3_joint3: axis 0 0 1 -> 0 1 0; limit lower=-0.4932 upper=1.6272 effort=0.3 velocity=12.863 -> lower=-0.4847 upper=1.5411 effort=0.2078 velocity=13.578; origin xyz=0.043618 0 -0.00475 rpy=1.5705 0 0 -> xyz=-0.00312502618421547 0.000100282625113788 0.0436176874508615 rpy=0 0 0.000268612717747223
- joint finger3_joint4: axis 0 0 1 -> 0 1 0; limit lower=-0.4932 upper=1.6272 effort=0.3 velocity=13.579 -> lower=-0.4671 upper=1.5788 effort=0.2018 velocity=12.863; origin xyz=0.0295 0 0 rpy=0 0 0 -> xyz=0 0 0.0294999999999998 rpy=0 0 0
- joint finger3_tip_fixed: origin xyz=0.0267 -0.0010501 0 rpy=0 0 0 -> xyz=-0.00199999998882053 -9.99999999926624E-05 0.0239466139625789 rpy=0 0 0
- joint finger4_joint1: axis 1 0 0 -> 0 1 0; limit lower=-0.32695 upper=1.63595 effort=1 velocity=8.203 -> lower=-0.1507 upper=1.5636 effort=0.6389 velocity=8.203; origin xyz=-0.0076649 0.013712 0.084429 rpy=-0.083776 0.090059 1.5161 -> xyz=-0.0076649 0.013712 0.084429 rpy=-0.090059 0 -0.054679
- joint finger4_joint2: axis 0 0 -1 -> -1 0 0; limit lower=-0.495 upper=0.495 effort=0.2 velocity=8.1158 -> lower=-0.4101 upper=0.3014 effort=0.1832 velocity=8.115; origin xyz=0 -0.0022 0.004 rpy=1.5708 -1.5708 0 -> xyz=0.000238272023819444 0 0.00403409169489746 rpy=0 -0.0837758044893524 0
- joint finger4_joint3: axis 0 0 1 -> 0 1 0; limit lower=-0.4932 upper=1.6272 effort=0.3 velocity=12.863 -> lower=-0.4747 upper=1.5526 effort=0.2249 velocity=13.578; origin xyz=0.043618 0 -0.00475 rpy=1.5705 0 0 -> xyz=-0.00312502629370909 0.000100282441161618 0.0436176874512648 rpy=0 0 0.000268623287696204
- joint finger4_joint4: axis 0 0 1 -> 0 1 0; limit lower=-0.4932 upper=1.6272 effort=0.3 velocity=13.579 -> lower=-0.4729 upper=1.5718 effort=0.2044 velocity=12.863; origin xyz=0.0295 0 0 rpy=0 0 0 -> xyz=0 0 0.0295000000000005 rpy=0 0 0
- joint finger4_tip_fixed: origin xyz=0.0267 -0.0010573 0 rpy=0 0 0 -> xyz=-0.00199999999999928 -9.99999794204474E-05 0.0239466139617312 rpy=0 0 0
- joint finger5_joint1: axis 1 0 0 -> 0 1 0; limit lower=-0.32695 upper=1.636 effort=1 velocity=8.203 -> lower=-0.1578 upper=1.5632 effort=0.6441 velocity=8.203; origin xyz=-0.0022687 0.034001 0.074281 rpy=-0.094248 0.19165 1.3951 -> xyz=-0.00226865105948153 0.0340011106647822 0.0742813381432918 rpy=-0.191650218499317 0 -0.175676455157885
- joint finger5_joint2: axis 0 0 -1 -> -1 0 0; limit lower=-0.495 upper=0.495 effort=0.2 velocity=8.1158 -> lower=-0.4103 upper=0.2949 effort=0.1798 velocity=8.115; origin xyz=0 -0.0022 0.004 rpy=-0.0067566 -1.5708 1.5776 -> xyz=0.000196015009673409 0 0.00403636545307588 rpy=0 -0.0942477800158131 0
- joint finger5_joint3: axis 0 0 1 -> 0 1 0; limit lower=-0.4932 upper=1.6272 effort=0.3 velocity=12.863 -> lower=-0.4733 upper=1.5560 effort=0.2384 velocity=13.578; origin xyz=0.043618 0 -0.00475 rpy=1.5705 0 0 -> xyz=-0.00312502637316564 0.000100282626826854 0.0436176864544762 rpy=0 0 0.000268612717748753
- joint finger5_joint4: axis 0 0 1 -> 0 1 0; limit lower=-0.4932 upper=1.6272 effort=0.3 velocity=13.579 -> lower=-0.4662 upper=1.5760 effort=0.1866 velocity=12.863; origin xyz=0.0295 0 0 rpy=0 0 0 -> xyz=0 0 0.0295000009963936 rpy=0 0 0
- joint finger5_tip_fixed: origin xyz=0.0267 -0.0010582 0 rpy=0 0 0 -> xyz=-0.00200000001120192 -9.99999794204162E-05 0.0239466139607956 rpy=0 0 0

File: wujihand_system/third_party/wuji_retargeting/wuji_retargeting/wuji_hand_description/urdf/right.urdf (robot description, URDF)
Before this commit: robot wujihand-right-v1.0.2, 26 links, 25 joints
Links:
- link finger1_link1: geometry collision mesh filename=finger1_link1.STL; visual mesh filename=finger1_link1.STL
- link finger1_link2: geometry collision mesh filename=finger1_link2.STL; visual mesh filename=finger1_link2.STL
- link finger1_link3: geometry collision mesh filename=finger1_link3.STL; visual mesh filename=finger1_link3.STL
- link finger1_link4: geometry collision mesh filename=finger1_link4.STL; visual mesh filename=finger1_link4.STL
- link finger1_tip_link: mass 0.004 -> 0.0041; geometry collision mesh filename=finger1_tip_link.STL; visual mesh filename=finger1_tip_link.STL
- link finger2_link1: geometry collision mesh filename=finger2_link1.STL; visual mesh filename=finger2_link1.STL
- link finger2_link2: geometry collision mesh filename=finger2_link2.STL; visual mesh filename=finger2_link2.STL
- link finger2_link3: geometry collision mesh filename=finger2_link3.STL; visual mesh filename=finger2_link3.STL
- link finger2_link4: geometry collision mesh filename=finger2_link4.STL; visual mesh filename=finger2_link4.STL
- link finger2_tip_link: mass 0.004 -> 0.00318; geometry collision mesh filename=finger2_tip_link.STL; visual mesh filename=finger2_tip_link.STL
- link finger3_link1: geometry collision mesh filename=finger3_link1.STL; visual mesh filename=finger3_link1.STL
- link finger3_link2: geometry collision mesh filename=finger3_link2.STL; visual mesh filename=finger3_link2.STL
- link finger3_link3: geometry collision mesh filename=finger3_link3.STL; visual mesh filename=finger3_link3.STL
- link finger3_link4: geometry collision mesh filename=finger3_link4.STL; visual mesh filename=finger3_link4.STL
- link finger3_tip_link: mass 0.004 -> 0.00318; geometry collision mesh filename=finger3_tip_link.STL; visual mesh filename=finger3_tip_link.STL
- link finger4_link1: geometry collision mesh filename=finger4_link1.STL; visual mesh filename=finger4_link1.STL
- link finger4_link2: geometry collision mesh filename=finger4_link2.STL; visual mesh filename=finger4_link2.STL
- link finger4_link3: geometry collision mesh filename=finger4_link3.STL; visual mesh filename=finger4_link3.STL
- link finger4_link4: geometry collision mesh filename=finger4_link4.STL; visual mesh filename=finger4_link4.STL
- link finger4_tip_link: mass 0.004 -> 0.00318; geometry collision mesh filename=finger4_tip_link.STL; visual mesh filename=finger4_tip_link.STL
- link finger5_link1: geometry collision mesh filename=finger5_link1.STL; visual mesh filename=finger5_link1.STL
- link finger5_link2: geometry collision mesh filename=finger5_link2.STL; visual mesh filename=finger5_link2.STL
- link finger5_link3: geometry collision mesh filename=finger5_link3.STL; visual mesh filename=finger5_link3.STL
- link finger5_link4: geometry collision mesh filename=finger5_link4.STL; visual mesh filename=finger5_link4.STL
- link finger5_tip_link: mass 0.004 -> 0.00318; geometry collision mesh filename=finger5_tip_link.STL; visual mesh filename=finger5_tip_link.STL
- link palm_link: mass 0.2179 -> 0.16914; geometry collision mesh filename=palm_link.STL; visual mesh filename=palm_link.STL
Joints:
- joint finger1_joint1: limit lower=-0.0448 upper=1.6508 effort=0.6 velocity=8.58701992 -> lower=0.0368 upper=1.6125 effort=0.4452 velocity=8.58701992
- joint finger1_joint2: limit lower=-0.1659 upper=0.9339 effort=0.6 velocity=11.10029404 -> lower=-0.1576 upper=0.9312 effort=0.4259 velocity=11.10029404
- joint finger1_joint3: limit lower=-0.4932 upper=1.6272 effort=0.3 velocity=12.86307659 -> lower=-0.4638 upper=1.5607 effort=0.1888 velocity=12.86307659
- joint finger1_joint4: limit lower=-0.4932 upper=1.6272 effort=0.3 velocity=13.57866158 -> lower=-0.4829 upper=1.5451 effort=0.1468 velocity=13.57866158
- joint finger2_joint1: limit lower=-0.32695 upper=1.63595 effort=1 velocity=8.203047484 -> lower=-0.1611 upper=1.5588 effort=0.6188 velocity=8.203047484
- joint finger2_joint2: limit lower=-0.495 upper=0.495 effort=0.2 velocity=8.115781022 -> lower=-0.4044 upper=0.3054 effort=0.1822 velocity=8.115781022
- joint finger2_joint3: limit lower=-0.4932 upper=1.6272 effort=0.3 velocity=12.86307659 -> lower=-0.4714 upper=1.5504 effort=0.2251 velocity=12.86307659
- joint finger2_joint4: limit lower=-0.4932 upper=1.6272 effort=0.3 velocity=13.57866158 -> lower=-0.4644 upper=1.5753 effort=0.2170 velocity=13.57866158
- joint finger3_joint1: limit lower=-0.32695 upper=1.63595 effort=1 velocity=8.203047484 -> lower=-0.1719 upper=1.5496 effort=0.6494 velocity=8.203047484
- joint finger3_joint2: limit lower=-0.495 upper=0.495 effort=0.2 velocity=8.115781022 -> lower=-0.4014 upper=0.2996 effort=0.1827 velocity=8.115781022
- joint finger3_joint3: limit lower=-0.4932 upper=1.6272 effort=0.3 velocity=12.86307659 -> lower=-0.4632 upper=1.5613 effort=0.2078 velocity=12.86307659
- joint finger3_joint4: limit lower=-0.4932 upper=1.6272 effort=0.3 velocity=13.57866158 -> lower=-0.4697 upper=1.5702 effort=0.2018 velocity=13.57866158
- joint finger4_joint1: limit lower=-0.32695 upper=1.63595 effort=1 velocity=8.203047484 -> lower=-0.1601 upper=1.5534 effort=0.6389 velocity=8.203047484
- joint finger4_joint2: limit lower=-0.495 upper=0.495 effort=0.2 velocity=8.115781022 -> lower=-0.4134 upper=0.3161 effort=0.1832 velocity=8.115781022
- joint finger4_joint3: limit lower=-0.4932 upper=1.6272 effort=0.3 velocity=12.86307659 -> lower=-0.4782 upper=1.5448 effort=0.2249 velocity=12.86307659
- joint finger4_joint4: limit lower=-0.4932 upper=1.6272 effort=0.3 velocity=13.57866158 -> lower=-0.4825 upper=1.5550 effort=0.2044 velocity=13.57866158
- joint finger5_joint1: limit lower=-0.32695 upper=1.63595 effort=1 velocity=8.203047484 -> lower=-0.1674 upper=1.5539 effort=0.6441 velocity=8.203047484
- joint finger5_joint2: limit lower=-0.495 upper=0.495 effort=0.2 velocity=8.115781022 -> lower=-0.4203 upper=0.2931 effort=0.1798 velocity=8.115781022
- joint finger5_joint3: limit lower=-0.4932 upper=1.6272 effort=0.3 velocity=12.86307659 -> lower=-0.4804 upper=1.5420 effort=0.2384 velocity=12.86307659
- joint finger5_joint4: limit lower=-0.4932 upper=1.6272 effort=0.3 velocity=13.57866158 -> lower=-0.4705 upper=1.5709 effort=0.1866 velocity=13.57866158
